Commit message: Add bottle demonstrations and medium ACT training with Gazebo rollout
Collect three-view RGB bottle pick-and-place demonstrations with local capture staging. Add fine-tuned ResNet18 ACT, fixed validation frames, configurable episode sampling, checkpoint resume, and live Gazebo inference. Include motion tools, documentation, and 100 passing unit tests.

File: src/robot_pick_place/kinova_gen3_lite_support/urdf/gen3_lite.urdf.xacro (robot description, xacro)
@@ -3,4 +3,5 @@
   <xacro:arg name="controllers_file" default="$(find kinova_gen3_lite_support)/config/ros2_controllers.yaml"/>
   <xacro:arg name="use_camera" default="false"/>
+  <xacro:arg name="use_demonstration_cameras" default="false"/>
   <xacro:include filename="$(find kortex_description)/robots/kortex_robot.xacro"/>
   <link name="world"/>
@@ -45,3 +46,36 @@
     </gazebo>
   </xacro:if>
+  <!-- Optional ACT collection views. The existing scene RGBD view stays unchanged. -->
+  <xacro:if value="$(arg use_demonstration_cameras)">
+    <xacro:macro name="demonstration_camera" params="name parent xyz rpy">
+      <link name="${name}_camera_link">
+        <inertial><mass value="0.001"/><inertia ixx="0.000001" ixy="0" ixz="0" iyy="0.000001" iyz="0" izz="0.000001"/></inertial>
+        <visual><geometry><box size="0.015 0.025 0.015"/></geometry>
+          <material name="${name}_camera_black"><color rgba="0.08 0.08 0.08 1"/></material>
+        </visual>
+      </link>
+      <joint name="${name}_camera_joint" type="fixed">
+        <parent link="${parent}"/><child link="${name}_camera_link"/>
+        <origin xyz="${xyz}" rpy="${rpy}"/>
+      </joint>
+      <gazebo reference="${name}_camera_link">
+        <sensor name="${name}_rgb" type="camera">
+          <topic>camera_${name}/image</topic><gz_frame_id>${name}_camera_link</gz_frame_id>
+          <always_on>true</always_on><update_rate>10</update_rate>
+          <camera>
+            <camera_info_topic>camera_${name}/camera_info</camera_info_topic>
+            <horizontal_fov>1.4</horizontal_fov>
+            <image><width>640</width><height>480</height><format>R8G8B8</format></image>
+            <clip><near>0.02</near><far>4.0</far></clip>
+          </camera>
+        </sensor>
+      </gazebo>
+    </xacro:macro>
+    <!-- Offset beside the palm, looking ahead toward the space between the fingers. -->
+    <xacro:demonstration_camera name="wrist" parent="gripper_base_link"
+      xyz="0.06 0 0.055" rpy="0 -0.89605538 3.14159265359"/>
+    <!-- Opposite oblique view covers both the tabletop and the bin. -->
+    <xacro:demonstration_camera name="side" parent="base_link"
+      xyz="1.0 0.4 0.7" rpy="0 0.593416 -2.475623"/>
+  </xacro:if>
 </robot>
